File: pcb/Si5351APicoBoB.sch (KiCad schematic (older format))
At the start: 11 parts

Commit message: Layout PCB, create rendering
Parts:
- removed J? (x3): CONN_01X02, symbol CONN_01X02
- added J3: CONN_01X06, Socket_Strips:Socket_Strip_Straight_1x06_Pitch2.54mm, symbol CONN_01X06
- C1, C2: renamed from C?; footprint (none) -> Capacitors_SMD:C_0603
- J1: renamed from J?; footprint (none) -> Socket_Strips:Socket_Strip_Straight_1x04_Pitch2.54mm
- J2: renamed from J?; footprint (none) -> EtherkitKicadLibrary:SMA-ENDLAUNCH
- R1, R2: renamed from R?; footprint (none) -> Resistors_SMD:R_0603
- U1: renamed from U?; value OSCILLATOR -> ASTX-H11-25.000MHZ-T; footprint (none) -> EtherkitKicadLibrary:ASTX-H11-25.000MHZ-T
- U2: renamed from U?; footprint MODULE -> EtherkitKicadLibrary:MSOP-10
Connections:
- net GND: now also J3.2 (P2), J3.4 (P4), J3.6 (P6)
- net at J2.1 (In), U2.10 (CLK0): now also J3.1 (P1)
- net at U2.6 (CLK2): now also J3.5 (P5)
- net at U2.9 (CLK1): now also J3.3 (P3)
Changed lines of the file:
@@
 LIBS:contrib
 LIBS:valves
+LIBS:Si5351APicoBoB-cache
 EELAYER 25 0
 EELAYER END
@@
 $EndDescr
 $Comp
-L SI5351A U?
+L SI5351A U2
 U 1 1 59498795
 P 5250 3750
-F 0 "U?" H 5250 4310 50  0000 C CNN
+F 0 "U2" H 5250 4310 50  0000 C CNN
 F 1 "SI5351A" H 5250 4225 50  0000 C CNN
-F 2 "MODULE" H 5250 3750 50  0001 C CNN
+F 2 "EtherkitKicadLibrary:MSOP-10" H 5250 3750 50  0001 C CNN
 F 3 "DOCUMENTATION" H 5250 3750 50  0001 C CNN
 	1    5250 3750
@@
 $EndComp
 $Comp
-L C C?
+L C C2
 U 1 1 59498A25
 P 4250 3100
-F 0 "C?" H 4400 3135 50  0000 C CNN
+F 0 "C2" H 4400 3135 50  0000 C CNN
 F 1 "100n" H 4450 3050 50  0000 C CNN
-F 2 "" H 4250 3100 60  0000 C CNN
+F 2 "Capacitors_SMD:C_0603" H 4250 3100 60  0001 C CNN
 F 3 "" H 4250 3100 60  0000 C CNN
 	1    4250 3100
@@
 $EndComp
 $Comp
-L C C?
+L C C1
 U 1 1 59498A4E
 P 3400 3450
-F 0 "C?" H 3550 3485 50  0000 C CNN
+F 0 "C1" H 3550 3485 50  0000 C CNN
 F 1 "100n" H 3600 3400 50  0000 C CNN
-F 2 "" H 3400 3450 60  0000 C CNN
+F 2 "Capacitors_SMD:C_0603" H 3400 3450 60  0001 C CNN
 F 3 "" H 3400 3450 60  0000 C CNN
 	1    3400 3450
@@
 $EndComp
 $Comp
-L R R?
+L R R1
 U 1 1 59498AED
 P 3350 4300
-F 0 "R?" H 3460 4340 50  0000 C CNN
+F 0 "R1" H 3460 4340 50  0000 C CNN
 F 1 "10k" H 3475 4250 50  0000 C CNN
-F 2 "" H 3350 4300 60  0000 C CNN
+F 2 "Resistors_SMD:R_0603" H 3350 4300 60  0001 C CNN
 F 3 "" H 3350 4300 60  0000 C CNN
 	1    3350 4300
@@
 $EndComp
 $Comp
-L R R?
+L R R2
 U 1 1 59498B22
 P 3650 4300
-F 0 "R?" H 3760 4340 50  0000 C CNN
+F 0 "R2" H 3760 4340 50  0000 C CNN
 F 1 "10k" H 3775 4250 50  0000 C CNN
-F 2 "" H 3650 4300 60  0000 C CNN
+F 2 "Resistors_SMD:R_0603" H 3650 4300 60  0001 C CNN
 F 3 "" H 3650 4300 60  0000 C CNN
 	1    3650 4300
@@
 $EndComp
 $Comp
-L BNC J?
+L BNC J2
 U 1 1 59498B6F
 P 6800 3550
-F 0 "J?" H 6800 3730 50  0000 C CNN
+F 0 "J2" H 6800 3730 50  0000 C CNN
 F 1 "SMA-END" H 6800 3660 50  0000 C CNN
-F 2 "" H 6800 3550 60  0000 C CNN
+F 2 "EtherkitKicadLibrary:SMA-ENDLAUNCH" H 6800 3550 60  0001 C CNN
 F 3 "" H 6800 3550 60  0000 C CNN
 	1    6800 3550
@@
 $EndComp
 $Comp
-L CONN_01X02 J?
-U 1 1 59498BCA
-P 7200 3600
-F 0 "J?" H 7200 3750 50  0000 C CNN
-F 1 "CONN_01X02" V 7300 3600 50  0001 C CNN
-F 2 "" H 7200 3600 50  0001 C CNN
-F 3 "" H 7200 3600 50  0001 C CNN
-	1    7200 3600
-	1    0    0    -1
-$EndComp
-$Comp
-L CONN_01X02 J?
-U 1 1 59498BF4
-P 7200 4050
-F 0 "J?" H 7200 4200 50  0000 C CNN
-F 1 "CONN_01X02" V 7300 4050 50  0001 C CNN
-F 2 "" H 7200 4050 50  0001 C CNN
-F 3 "" H 7200 4050 50  0001 C CNN
-	1    7200 4050
-	1    0    0    -1
-$EndComp
-$Comp
-L CONN_01X02 J?
-U 1 1 59498C2E
-P 7200 4450
-F 0 "J?" H 7200 4600 50  0000 C CNN
-F 1 "CONN_01X02" V 7300 4450 50  0001 C CNN
-F 2 "" H 7200 4450 50  0001 C CNN
-F 3 "" H 7200 4450 50  0001 C CNN
-	1    7200 4450
-	1    0    0    -1
-$EndComp
-$Comp
-L OSCILLATOR U?
+L OSCILLATOR U1
 U 1 1 59498CCB
 P 4100 3650
-F 0 "U?" H 3650 4300 50  0000 C CNN
-F 1 "OSCILLATOR" H 3800 4150 50  0000 C CNN
-F 2 "" H 4100 3650 60  0000 C CNN
+F 0 "U1" H 4025 4175 50  0000 C CNN
+F 1 "ASTX-H11-25.000MHZ-T" H 3575 4075 50  0000 C CNN
+F 2 "EtherkitKicadLibrary:ASTX-H11-25.000MHZ-T" H 4100 3650 60  0001 C CNN
 F 3 "" H 4100 3650 60  0000 C CNN
 	1    4100 3650
@@
 $EndComp
 $Comp
-L CONN_01X04 J?
+L CONN_01X04 J1
 U 1 1 59498DCA
 P 2600 4400
-F 0 "J?" H 2600 4650 50  0000 C CNN
+F 0 "J1" H 2600 4650 50  0000 C CNN
 F 1 "CONN_01X04" V 2700 4400 50  0001 C CNN
-F 2 "" H 2600 4400 50  0001 C CNN
+F 2 "Socket_Strips:Socket_Strip_Straight_1x04_Pitch2.54mm" H 2600 4400 50  0001 C CNN
 F 3 "" H 2600 4400 50  0001 C CNN
 	1    2600 4400
@@
 $EndComp
 $Comp
-L GND #PWR?
+L GND #PWR4
 U 1 1 59498EDF
 P 4100 3900
-F 0 "#PWR?" H 4100 3650 50  0001 C CNN
+F 0 "#PWR4" H 4100 3650 50  0001 C CNN
 F 1 "GND" H 4100 3750 50  0000 C CNN
 F 2 "" H 4100 3900 50  0001 C CNN
@@
 $EndComp
 $Comp
-L GND #PWR?
+L GND #PWR3
 U 1 1 59498F12
 P 3400 3550
-F 0 "#PWR?" H 3400 3300 50  0001 C CNN
+F 0 "#PWR3" H 3400 3300 50  0001 C CNN
 F 1 "GND" H 3400 3400 50  0000 C CNN
 F 2 "" H 3400 3550 50  0001 C CNN
@@
 $EndComp
 $Comp
-L GND #PWR?
+L GND #PWR6
 U 1 1 59498F3E
 P 4250 3200
-F 0 "#PWR?" H 4250 2950 50  0001 C CNN
+F 0 "#PWR6" H 4250 2950 50  0001 C CNN
 F 1 "GND" H 4250 3050 50  0000 C CNN
 F 2 "" H 4250 3200 50  0001 C CNN
@@
 $EndComp
 $Comp
-L GND #PWR?
+L GND #PWR9
 U 1 1 59498F6A
 P 6800 3700
-F 0 "#PWR?" H 6800 3450 50  0001 C CNN
+F 0 "#PWR9" H 6800 3450 50  0001 C CNN
 F 1 "GND" H 6800 3550 50  0000 C CNN
 F 2 "" H 6800 3700 50  0001 C CNN
@@
 $EndComp
 $Comp
-L GND #PWR?
+L GND #PWR12
 U 1 1 59498FC2
-P 7000 4100
-F 0 "#PWR?" H 7000 3850 50  0001 C CNN
-F 1 "GND" H 7000 3950 50  0000 C CNN
-F 2 "" H 7000 4100 50  0001 C CNN
-F 3 "" H 7000 4100 50  0001 C CNN
-	1    7000 4100
-	1    0    0    -1
-$EndComp
-$Comp
-L GND #PWR?
+P 7450 4050
+F 0 "#PWR12" H 7450 3800 50  0001 C CNN
+F 1 "GND" H 7450 3900 50  0000 C CNN
+F 2 "" H 7450 4050 50  0001 C CNN
+F 3 "" H 7450 4050 50  0001 C CNN
+	1    7450 4050
+	1    0    0    -1
+$EndComp
+$Comp
+L GND #PWR11
 U 1 1 59498FEE
-P 7000 4500
-F 0 "#PWR?" H 7000 4250 50  0001 C CNN
-F 1 "GND" H 7000 4350 50  0000 C CNN
-F 2 "" H 7000 4500 50  0001 C CNN
-F 3 "" H 7000 4500 50  0001 C CNN
-	1    7000 4500
-	1    0    0    -1
-$EndComp
-$Comp
-L GND #PWR?
+P 7200 3850
+F 0 "#PWR11" H 7200 3600 50  0001 C CNN
+F 1 "GND" H 7200 3700 50  0000 C CNN
+F 2 "" H 7200 3850 50  0001 C CNN
+F 3 "" H 7200 3850 50  0001 C CNN
+	1    7200 3850
+	1    0    0    -1
+$EndComp
+$Comp
+L GND #PWR2
 U 1 1 5949905C
 P 2800 4550
-F 0 "#PWR?" H 2800 4300 50  0001 C CNN
+F 0 "#PWR2" H 2800 4300 50  0001 C CNN
 F 1 "GND" H 2800 4400 50  0000 C CNN
 F 2 "" H 2800 4550 50  0001 C CNN
@@
 $EndComp
 $Comp
-L +3.3V #PWR?
+L +3.3V #PWR5
 U 1 1 594990D7
 P 4250 2900
-F 0 "#PWR?" H 4250 2860 30  0001 C CNN
+F 0 "#PWR5" H 4250 2860 30  0001 C CNN
 F 1 "+3.3V" H 4250 3010 50  0000 C CNN
 F 2 "" H 4250 2900 60  0000 C CNN
@@
 $EndComp
 $Comp
-L +3.3V #PWR?
+L +3.3V #PWR1
 U 1 1 5949910A
 P 2800 4000
-F 0 "#PWR?" H 2800 3960 30  0001 C CNN
+F 0 "#PWR1" H 2800 3960 30  0001 C CNN
 F 1 "+3.3V" H 2800 4110 50  0000 C CNN
 F 2 "" H 2800 4000 60  0000 C CNN
@@
 	4600 3850 4400 3850
 Wire Wire Line
-	4400 4500 4400 3850
-Wire Wire Line
-	3100 4500 4400 4500
+	4400 3850 4400 4500
+Wire Wire Line
+	4400 4500 3100 4500
 Wire Wire Line
 	3100 4500 3100 4350
@@
 	4600 3950 4450 3950
 Wire Wire Line
-	4450 4600 4450 3950
-Wire Wire Line
-	3000 4600 4450 4600
+	4450 3950 4450 4600
+Wire Wire Line
+	4450 4600 3000 4600
 Wire Wire Line
 	3000 4600 3000 4450
@@
 Connection ~ 3750 3300
 $Comp
-L GND #PWR?
+L GND #PWR7
 U 1 1 594993D2
 P 6050 3750
-F 0 "#PWR?" H 6050 3500 50  0001 C CNN
+F 0 "#PWR7" H 6050 3500 50  0001 C CNN
 F 1 "GND" H 6100 3800 50  0000 C CNN
 F 2 "" H 6050 3750 50  0001 C CNN
@@
 $EndComp
 $Comp
-L +3.3V #PWR?
+L +3.3V #PWR8
 U 1 1 59499409
 P 6250 3900
-F 0 "#PWR?" H 6250 3860 30  0001 C CNN
+F 0 "#PWR8" H 6250 3860 30  0001 C CNN
 F 1 "+3.3V" H 6250 4010 50  0000 C CNN
 F 2 "" H 6250 3900 60  0000 C CNN
@@
 	6800 3700 6800 3700
 Wire Wire Line
-	7000 4000 6550 4000
+	6550 4000 7100 4000
 Wire Wire Line
 	6550 4000 6550 3650
 Wire Wire Line
 	6550 3650 5900 3650
-Wire Wire Line
-	7000 4400 5900 4400
-Wire Wire Line
-	5900 4400 5900 3950
-$Comp
-L GND #PWR?
+$Comp
+L GND #PWR10
 U 1 1 5949967F
 P 7000 3700
-F 0 "#PWR?" H 7000 3450 50  0001 C CNN
+F 0 "#PWR10" H 7000 3450 50  0001 C CNN
 F 1 "GND" H 7000 3550 50  0000 C CNN
 F 2 "" H 7000 3700 50  0001 C CNN
@@
 $EndComp
 NoConn ~ 4600 3750
+$Comp
+L CONN_01X06 J3
+U 1 1 594E9591
+P 7650 3800
+F 0 "J3" H 7650 4150 50  0000 C CNN
+F 1 "CONN_01X06" V 7750 3800 50  0001 C CNN
+F 2 "Socket_Strips:Socket_Strip_Straight_1x06_Pitch2.54mm" H 7650 3800 50  0001 C CNN
+F 3 "" H 7650 3800 50  0001 C CNN
+	1    7650 3800
+	1    0    0    -1
+$EndComp
+Wire Wire Line
+	7000 3550 7450 3550
+Wire Wire Line
+	7100 4000 7100 3750
+Wire Wire Line
+	7100 3750 7450 3750
+Wire Wire Line
+	7000 3650 7450 3650
+Wire Wire Line
+	7200 3850 7450 3850
+Wire Wire Line
+	5900 3950 6475 3950
+Wire Wire Line
+	6475 3950 6475 4075
+Wire Wire Line
+	6475 4075 7350 4075
+Wire Wire Line
+	7350 4075 7350 3950
+Wire Wire Line
+	7350 3950 7450 3950
 $EndSCHEMATC
